File: rcj_res_b_board.kicad_pcb (KiCad board)
At the start: 2 copper layers, 92.5 x 100 mm, 93 parts, among them P1 GP2Y0A41SK0F, P10 SERVO0, P11 MPU9250, P12 PING0, P13 CONN_01X03, P14 CONN_01X03, P15 CONN_01X04, P16 CONN_02X04, P2 GP2Y0A41SK0F, P3 GP2Y0A41SK0F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

Commit message: Changed resistor value
Changed value on phototransistor of light sensor to get higher dynamic range in readings
	(tested)
Parts:
- R11: value 1k -> 10k
Connections:
- MCU1 pad 1: (no net) -> Net-(MCU1-Pad1)
- MCU1 pad 15: (no net) -> Net-(MCU1-Pad15)
- MCU1 pad 2: (no net) -> Net-(MCU1-Pad2)
- MCU1 pad 20: (no net) -> Net-(MCU1-Pad20)
- MCU1 pad 36: (no net) -> Net-(MCU1-Pad36)
- MCU1 pad 40: (no net) -> Net-(MCU1-Pad40)
- MCU1 pad 5: (no net) -> Net-(MCU1-Pad5)
- MCU1 pad 53: (no net) -> Net-(MCU1-Pad53)
- MCU1 pad 56: (no net) -> Net-(MCU1-Pad56)
- MCU1 pad 6: (no net) -> Net-(MCU1-Pad6)
- MCU1 pad 62: (no net) -> Net-(MCU1-Pad62)
- P16 pad 8: (no net) -> Net-(P16-Pad8)
- P_CT1 pad 8: (no net) -> Net-(P_CT1-Pad8)
- REG1 pad 4: (no net) -> Net-(REG1-Pad4)
Changed lines of the file:
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@@
-(kicad_pcb (version 4) (host pcbnew 0.201512311516+6410~40~ubuntu15.04.1-stable)
+(kicad_pcb (version 4) (host pcbnew 0.201601310801+6528~42~ubuntu15.04.1-product)
   (general
     (links 227)
@@
     (zones 0)
     (modules 93)
-    (nets 82)
+    (nets 96)
   )
   (page A4)
@@
   (net 80 /OLED_Circuitry/MOSI)
   (net 81 "Net-(P_BAT1-Pad2)")
+  (net 82 "Net-(MCU1-Pad1)")
+  (net 83 "Net-(MCU1-Pad2)")
+  (net 84 "Net-(MCU1-Pad5)")
+  (net 85 "Net-(MCU1-Pad6)")
+  (net 86 "Net-(MCU1-Pad15)")
+  (net 87 "Net-(MCU1-Pad20)")
+  (net 88 "Net-(MCU1-Pad36)")
+  (net 89 "Net-(MCU1-Pad40)")
+  (net 90 "Net-(MCU1-Pad53)")
+  (net 91 "Net-(MCU1-Pad56)")
+  (net 92 "Net-(MCU1-Pad62)")
+  (net 93 "Net-(P16-Pad8)")
+  (net 94 "Net-(P_CT1-Pad8)")
+  (net 95 "Net-(REG1-Pad4)")
   (net_class Default "This is the default net class."
     (clearance 0.15)
@@
     (add_net "Net-(D3-Pad2)")
     (add_net "Net-(D4-Pad2)")
+    (add_net "Net-(MCU1-Pad1)")
+    (add_net "Net-(MCU1-Pad15)")
+    (add_net "Net-(MCU1-Pad2)")
+    (add_net "Net-(MCU1-Pad20)")
+    (add_net "Net-(MCU1-Pad36)")
+    (add_net "Net-(MCU1-Pad40)")
+    (add_net "Net-(MCU1-Pad5)")
+    (add_net "Net-(MCU1-Pad53)")
+    (add_net "Net-(MCU1-Pad56)")
+    (add_net "Net-(MCU1-Pad6)")
+    (add_net "Net-(MCU1-Pad62)")
     (add_net "Net-(OLED1-Pad13)")
+    (add_net "Net-(P16-Pad8)")
+    (add_net "Net-(P_CT1-Pad8)")
     (add_net "Net-(R9-Pad2)")
+    (add_net "Net-(REG1-Pad4)")
     (add_net "Net-(SW3-Pad3)")
   )
@@
     (fp_line (start 5.175 5.175) (end 4.1 5.175) (layer B.SilkS) (width 0.15))
     (fp_line (start -5.175 4.1) (end -6.2 4.1) (layer B.SilkS) (width 0.15))
-    (pad 1 smd rect (at -5.7 3.75) (size 1 0.25) (layers B.Cu B.Paste B.Mask))
-    (pad 2 smd rect (at -5.7 3.25) (size 1 0.25) (layers B.Cu B.Paste B.Mask))
+    (pad 1 smd rect (at -5.7 3.75) (size 1 0.25) (layers B.Cu B.Paste B.Mask)
+      (net 82 "Net-(MCU1-Pad1)"))
+    (pad 2 smd rect (at -5.7 3.25) (size 1 0.25) (layers B.Cu B.Paste B.Mask)
+      (net 83 "Net-(MCU1-Pad2)"))
     (pad 3 smd rect (at -5.7 2.75) (size 1 0.25) (layers B.Cu B.Paste B.Mask)
       (net 65 /LED_USR1))
     (pad 4 smd rect (at -5.7 2.25) (size 1 0.25) (layers B.Cu B.Paste B.Mask)
       (net 66 /LED_USR2))
-    (pad 5 smd rect (at -5.7 1.75) (size 1 0.25) (layers B.Cu B.Paste B.Mask))
-    (pad 6 smd rect (at -5.7 1.25) (size 1 0.25) (layers B.Cu B.Paste B.Mask))
+    (pad 5 smd rect (at -5.7 1.75) (size 1 0.25) (layers B.Cu B.Paste B.Mask)
+      (net 84 "Net-(MCU1-Pad5)"))
+    (pad 6 smd rect (at -5.7 1.25) (size 1 0.25) (layers B.Cu B.Paste B.Mask)
+      (net 85 "Net-(MCU1-Pad6)"))
     (pad 7 smd rect (at -5.7 0.75) (size 1 0.25) (layers B.Cu B.Paste B.Mask)
       (net 61 "Net-(C22-Pad1)"))
@@
     (pad 14 smd rect (at -5.7 -2.75) (size 1 0.25) (layers B.Cu B.Paste B.Mask)
       (net 39 /TEMP1_PWM))
-    (pad 15 smd rect (at -5.7 -3.25) (size 1 0.25) (layers B.Cu B.Paste B.Mask))
+    (pad 15 smd rect (at -5.7 -3.25) (size 1 0.25) (layers B.Cu B.Paste B.Mask)
+      (net 86 "Net-(MCU1-Pad15)"))
     (pad 16 smd rect (at -5.7 -3.75) (size 1 0.25) (layers B.Cu B.Paste B.Mask)
       (net 29 /MD_APWM))
@@
     (pad 19 smd rect (at -2.75 -5.7 270) (size 1 0.25) (layers B.Cu B.Paste B.Mask)
       (net 3 /3.3V))
-    (pad 20 smd rect (at -2.25 -5.7 270) (size 1 0.25) (layers B.Cu B.Paste B.Mask))
+    (pad 20 smd rect (at -2.25 -5.7 270) (size 1 0.25) (layers B.Cu B.Paste B.Mask)
+      (net 87 "Net-(MCU1-Pad20)"))
     (pad 21 smd rect (at -1.75 -5.7 270) (size 1 0.25) (layers B.Cu B.Paste B.Mask)
       (net 14 /IR_L_F))
@@
     (pad 35 smd rect (at 5.7 -2.75) (size 1 0.25) (layers B.Cu B.Paste B.Mask)
       (net 25 /PING0_ECHO))
-    (pad 36 smd rect (at 5.7 -2.25) (size 1 0.25) (layers B.Cu B.Paste B.Mask))
+    (pad 36 smd rect (at 5.7 -2.25) (size 1 0.25) (layers B.Cu B.Paste B.Mask)
+      (net 88 "Net-(MCU1-Pad36)"))
     (pad 37 smd rect (at 5.7 -1.75) (size 1 0.25) (layers B.Cu B.Paste B.Mask)
       (net 7 /M0_ENC_A))
@@
     (pad 39 smd rect (at 5.7 -0.75) (size 1 0.25) (layers B.Cu B.Paste B.Mask)
       (net 26 /PING0_TRIG))
-    (pad 40 smd rect (at 5.7 -0.25) (size 1 0.25) (layers B.Cu B.Paste B.Mask))
+    (pad 40 smd rect (at 5.7 -0.25) (size 1 0.25) (layers B.Cu B.Paste B.Mask)
+      (net 89 "Net-(MCU1-Pad40)"))
     (pad 41 smd rect (at 5.7 0.25) (size 1 0.25) (layers B.Cu B.Paste B.Mask)
       (net 32 /MD_AIN1))
@@
     (pad 52 smd rect (at 2.25 5.7 270) (size 1 0.25) (layers B.Cu B.Paste B.Mask)
       (net 38 /UART_RX))
-    (pad 53 smd rect (at 1.75 5.7 270) (size 1 0.25) (layers B.Cu B.Paste B.Mask))
+    (pad 53 smd rect (at 1.75 5.7 270) (size 1 0.25) (layers B.Cu B.Paste B.Mask)
+      (net 90 "Net-(MCU1-Pad53)"))
     (pad 54 smd rect (at 1.25 5.7 270) (size 1 0.25) (layers B.Cu B.Paste B.Mask)
       (net 41 /OLED_SS))
     (pad 55 smd rect (at 0.75 5.7 270) (size 1 0.25) (layers B.Cu B.Paste B.Mask)
       (net 74 /SCLK))
-    (pad 56 smd rect (at 0.25 5.7 270) (size 1 0.25) (layers B.Cu B.Paste B.Mask))
+    (pad 56 smd rect (at 0.25 5.7 270) (size 1 0.25) (layers B.Cu B.Paste B.Mask)
+      (net 91 "Net-(MCU1-Pad56)"))
     (pad 57 smd rect (at -0.25 5.7 270) (size 1 0.25) (layers B.Cu B.Paste B.Mask)
       (net 75 /MOSI))
@@
     (pad 61 smd rect (at -2.25 5.7 270) (size 1 0.25) (layers B.Cu B.Paste B.Mask)
       (net 28 /SERVO0_PWM))
-    (pad 62 smd rect (at -2.75 5.7 270) (size 1 0.25) (layers B.Cu B.Paste B.Mask))
+    (pad 62 smd rect (at -2.75 5.7 270) (size 1 0.25) (layers B.Cu B.Paste B.Mask)
+      (net 92 "Net-(MCU1-Pad62)"))
     (pad 63 smd rect (at -3.25 5.7 270) (size 1 0.25) (layers B.Cu B.Paste B.Mask)
       (net 2 GNDD))
@@
       (effects (font (size 1 1) (thickness 0.15)) (justify mirror))
     )
-    (fp_text value 1k (at 0 -2) (layer B.Fab)
+    (fp_text value 10k (at 0 -2) (layer B.Fab)
       (effects (font (size 1 1) (thickness 0.15)) (justify mirror))
     )
@@
     (pad 3 smd rect (at -1.34 -0.95) (size 0.63 0.45) (layers B.Cu B.Paste B.Mask)
       (net 2 GNDD))
-    (pad 4 smd rect (at 1.34 -0.95) (size 0.63 0.45) (layers B.Cu B.Paste B.Mask))
+    (pad 4 smd rect (at 1.34 -0.95) (size 0.63 0.45) (layers B.Cu B.Paste B.Mask)
+      (net 95 "Net-(REG1-Pad4)"))
     (pad 5 smd rect (at 1.34 0) (size 0.63 0.45) (layers B.Cu B.Paste B.Mask)
       (net 59 /VBAT1))
@@
     (pad 7 thru_hole oval (at 7.62 0) (size 1.7272 1.7272) (drill 1.016) (layers *.Cu *.Mask F.SilkS)
       (net 42 /OLED_RST))
-    (pad 8 thru_hole oval (at 7.62 2.54) (size 1.7272 1.7272) (drill 1.016) (layers *.Cu *.Mask F.SilkS))
+    (pad 8 thru_hole oval (at 7.62 2.54) (size 1.7272 1.7272) (drill 1.016) (layers *.Cu *.Mask F.SilkS)
+      (net 93 "Net-(P16-Pad8)"))
     (model Socket_Strips.3dshapes/Socket_Strip_Straight_2x04.wrl
       (at (xyz 0.15 -0.05 0))
@@
     (pad 7 thru_hole oval (at 0 -7.62) (size 1.7272 1.7272) (drill 1.016) (layers *.Cu *.Mask B.SilkS)
       (net 77 /OLED_Circuitry/RST))
-    (pad 8 thru_hole oval (at 2.54 -7.62) (size 1.7272 1.7272) (drill 1.016) (layers *.Cu *.Mask B.SilkS))
+    (pad 8 thru_hole oval (at 2.54 -7.62) (size 1.7272 1.7272) (drill 1.016) (layers *.Cu *.Mask B.SilkS)
+      (net 94 "Net-(P_CT1-Pad8)"))
     (model Pin_Headers.3dshapes/Pin_Header_Straight_2x04.wrl
       (at (xyz 0.05 -0.15 0))

Commit message: Change resistor value
80 ohm resistor for floor light sensor was replaced by 100 ohm on boards, update schematics to match
Parts:
- R9: value 80 -> 100
Changed lines of the file:
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@@
-(kicad_pcb (version 4) (host pcbnew 0.201601310801+6528~42~ubuntu15.04.1-product)
+(kicad_pcb (version 20160815) (host pcbnew 4.1.0-alpha+201608181240+7066~46~ubuntu16.04.1-product)
   (general
     (links 227)
     (no_connects 0)
-    (area 19.924999 49.924999 112.575001 150.100001)
+    (area 18.9925 28.3 176.714287 188.100001)
     (thickness 1.6)
     (drawings 51)
@@
       (hpglpenspeed 20)
       (hpglpendiameter 15)
-      (hpglpenoverlay 2)
       (psnegative false)
       (psa4output false)
@@
     (uvia_dia 0.3)
     (uvia_drill 0.1)
+    (diff_pair_gap 0.25)
+    (diff_pair_width 0.2)
     (add_net /I2C_SCL)
     (add_net /I2C_SDA)
@@
     (uvia_dia 0.7)
     (uvia_drill 0.5)
+    (diff_pair_gap 0.25)
+    (diff_pair_width 0.2)
     (add_net /VBAT1)
     (add_net "Net-(NT2-Pad2)")
@@
     (uvia_dia 0.3)
     (uvia_drill 0.1)
+    (diff_pair_gap 0.25)
+    (diff_pair_width 0.2)
     (add_net /3.3V)
     (add_net /OLED_Circuitry/3.3V)
@@
     (uvia_dia 1.2)
     (uvia_drill 1)
+    (diff_pair_gap 0.25)
+    (diff_pair_width 0.2)
     (add_net GND)
     (add_net GNDPWR)
@@
     (uvia_dia 0.7)
     (uvia_drill 0.5)
+    (diff_pair_gap 0.25)
+    (diff_pair_width 0.2)
     (add_net "Net-(C1-Pad1)")
     (add_net "Net-(C1-Pad2)")
@@
     (descr "Through hole socket strip")
     (tags "socket strip")
-    (fp_text reference P9 (at -2.5 0 360) (layer B.SilkS)
+    (fp_text reference P9 (at -2.5 0) (layer B.SilkS)
       (effects (font (size 1 1) (thickness 0.15)) (justify mirror))
     )
-    (fp_text value CONN_01X02 (at 5 0 360) (layer B.Fab)
+    (fp_text value CONN_01X02 (at 5 0) (layer B.Fab)
       (effects (font (size 1 1) (thickness 0.15)) (justify mirror))
     )
@@
     (descr "Through hole socket strip")
     (tags "socket strip")
-    (fp_text reference P8 (at -2.5 0 360) (layer B.SilkS)
+    (fp_text reference P8 (at -2.5 0) (layer B.SilkS)
       (effects (font (size 1 1) (thickness 0.15)) (justify mirror))
     )
@@
     (tags SOT-23)
     (attr smd)
-    (fp_text reference HAL_M0A1 (at 2.25 -1 360) (layer B.SilkS)
+    (fp_text reference HAL_M0A1 (at 2.25 -1) (layer B.SilkS)
       (effects (font (size 1 1) (thickness 0.15)) (justify mirror))
     )
@@
     (tags SOT-23)
     (attr smd)
-    (fp_text reference HAL_M0B1 (at -2.25 -1 360) (layer B.SilkS)
+    (fp_text reference HAL_M0B1 (at -2.25 -1) (layer B.SilkS)
       (effects (font (size 1 1) (thickness 0.15)) (justify mirror))
     )
@@
     (descr "Through hole socket strip")
     (tags "socket strip")
-    (fp_text reference P7 (at -3 0 450) (layer F.SilkS)
+    (fp_text reference P7 (at -3 0 90) (layer F.SilkS)
       (effects (font (size 1 1) (thickness 0.15)))
     )
@@
       (effects (font (size 1 1) (thickness 0.15)) (justify mirror))
     )
-    (fp_text value 80 (at -0.05 2 180) (layer B.Fab)
+    (fp_text value 100 (at -0.05 2 180) (layer B.Fab)
       (effects (font (size 1 1) (thickness 0.15)) (justify mirror))
     )
@@
     (tags "capacitor 0805")
     (attr smd)
-    (fp_text reference C4 (at -2.5 0 360) (layer F.SilkS)
+    (fp_text reference C4 (at -2.5 0) (layer F.SilkS)
       (effects (font (size 1 1) (thickness 0.15)))
     )
@@
     (tags "capacitor 0805")
     (attr smd)
-    (fp_text reference C5 (at -2.5 0 360) (layer F.SilkS)
+    (fp_text reference C5 (at -2.5 0) (layer F.SilkS)
       (effects (font (size 1 1) (thickness 0.15)))
     )
@@
     (tags SOD-323)
     (attr smd)
-    (fp_text reference D1 (at -2.5 0 360) (layer F.SilkS)
+    (fp_text reference D1 (at -2.5 0) (layer F.SilkS)
       (effects (font (size 1 1) (thickness 0.15)))
     )
@@
     (tags "resistor 0805")
     (attr smd)
-    (fp_text reference R6 (at -2.5 0 360) (layer F.SilkS)
+    (fp_text reference R6 (at -2.5 0) (layer F.SilkS)
       (effects (font (size 1 1) (thickness 0.15)))
     )
@@
     (tags "capacitor 0805")
     (attr smd)
-    (fp_text reference C13 (at 3 0 360) (layer B.SilkS)
+    (fp_text reference C13 (at 3 0) (layer B.SilkS)
       (effects (font (size 1 1) (thickness 0.15)) (justify mirror))
     )
@@
   (module Custom:UG-2832HSWEG04 placed (layer B.Cu)
     (at 106 146 90)
-    (fp_text reference OLED1 (at -2 0 360) (layer B.SilkS)
+    (fp_text reference OLED1 (at -2 0) (layer B.SilkS)
       (effects (font (size 1 1) (thickness 0.15)) (justify mirror))
     )
-    (fp_text value UG-2832HSWEG04 (at 2 0 360) (layer B.Fab)
+    (fp_text value UG-2832HSWEG04 (at 2 0) (layer B.Fab)
       (effects (font (size 1 1) (thickness 0.15)) (justify mirror))
     )
@@
     (tags "resistor 0805")
     (attr smd)
-    (fp_text reference SB2 (at 2.5 0 360) (layer F.SilkS)
+    (fp_text reference SB2 (at 2.5 0) (layer F.SilkS)
       (effects (font (size 1 1) (thickness 0.15)))
     )
